Commit message: another set of typos

File: description/robot_core.xacro (robot description, xacro)
@@ -35,8 +35,8 @@
         </link>
     <!--Left Wheel-->
-        <joint name="left_wheel_joint" type="continuious">
+        <joint name="left_wheel_joint" type="continuous">
             <parent link="base_link"/>
             <child link="left_wheel"/>
-            <origin xyz="0 0.175 0" rpy="-$(pi/2) 0 0"/>
+            <origin xyz="0 0.175 0" rpy="$(xacro:math('-pi/2')) 0 0"/>
             <axis xyz="0 0 1"/>
         </joint>
@@ -58,8 +58,8 @@
         </link>
     <!--Right Wheel-->
-        <joint name="right_wheel_joint" type="continuious">
+        <joint name="right_wheel_joint" type="continuous">
             <parent link="base_link"/>
             <child link="right_wheel"/>
-            <origin xyz="0 -0.175 0" rpy="$(pi/2) 0 0"/>
+            <origin xyz="0 -0.175 0" rpy="$(xacro:math('pi/2')) 0 0"/>
             <axis xyz="0 0 -1"/>
         </joint>
@@ -86,8 +86,8 @@
             <origin xyz="0.24 0 0"/>
         </joint>
-        <link name="right_wheel">
+        <link name="caster_wheel">
             <visual>
                 <geometry>
-                    <shpere radius="0.05"/>
+                    <sphere radius="0.05"/>
                 </geometry>
                 <material name ="black"/>

Commit message: i hate everything

File: description/robot_core.xacro (robot description, xacro)
@@ -38,5 +38,5 @@
             <parent link="base_link"/>
             <child link="left_wheel"/>
-            <origin xyz="0 0.175 0" rpy="$(xacro:math('-pi/2')) 0 0"/>
+            <origin xyz="0 0.175 0" rpy="${-pi/2} 0 0"/>
             <axis xyz="0 0 1"/>
         </joint>
@@ -61,5 +61,5 @@
             <parent link="base_link"/>
             <child link="right_wheel"/>
-            <origin xyz="0 -0.175 0" rpy="$(xacro:math('pi/2')) 0 0"/>
+            <origin xyz="0 -0.175 0" rpy="${pi/2} 0 0"/>
             <axis xyz="0 0 -1"/>
         </joint>

Commit message: chat thinks transmission will fix problems

File: description/robot_core.xacro (robot description, xacro)
@@ -80,4 +80,24 @@
             </xacro:inertial_cylinder>
         </link>
+        <transmission name="left_wheel_trans">
+            <type>transmission_interface/SimpleTransmission</type>
+            <joint name="left_wheel_joint">
+                <hardwareInterface>velocity</hardwareInterface>
+            </joint>
+            <actuator name="left_wheel_motor">
+                <hardwareInterface>velocity</hardwareInterface>
+                <mechanicalReduction>1</mechanicalReduction>
+            </actuator>
+        </transmission>
+        <transmission name="right_wheel_trans">
+            <type>transmission_interface/SimpleTransmission</type>
+            <joint name="right_wheel_joint">
+                <hardwareInterface>velocity</hardwareInterface>
+            </joint>
+            <actuator name="right_wheel_motor">
+                <hardwareInterface>velocity</hardwareInterface>
+                <mechanicalReduction>1</mechanicalReduction>
+            </actuator>
+        </transmission>
     <!--castor wheel-->
         <joint name="caster_wheel_joint" type="fixed">
