Commit message: inertia also cant equal 0. also ajdusted plugin name

File: description/gazebo_control.xacro (robot description, xacro)
@@ -3,5 +3,5 @@
 <xacro:property name="body_color" value="Gazebo/Silver" />
 <gazebo>
-  <plugin name="control" filename="libgazebo_ros_control.so"/>
+  <plugin name="ignition::gazebo::systems::DiffDrive" filename="libignition-gazebo6-diff-drive-system.so"/>
 </gazebo>
 <gazebo reference="base_link">

File: description/robot.urdf.xacro (robot description, xacro)
@@ -8,5 +8,5 @@
     <origin xyz="0.0 0.0 0.0" rpy="0 0 0"/>
     <mass value="0.00001"/>
-    <inertia ixx="0.0" iyy="0.0" izz="0.0" ixy="0.0" iyz="0.0" ixz="0.0"/>
+    <inertia ixx="0.00001" iyy="0.00001" izz="0.00001" ixy="0.00001" iyz="0.00001" ixz="0.00001"/>
   </inertial>
   <visual>
