Commit message: updated package names and renamed duplicate links

File: description/robot.urdf.xacro (robot description, xacro)
@@ -13,5 +13,5 @@
     <origin xyz="0 0 0" rpy="0 0 0"/>
     <geometry>
-      <mesh filename="package://URDF_description/meshes/base_link.stl" scale="0.001 0.001 0.001"/>
+      <mesh filename="package://my_bot/meshes/base_link.stl" scale="0.001 0.001 0.001"/>
     </geometry>
     <material name="silver"/>
@@ -20,5 +20,5 @@
     <origin xyz="0 0 0" rpy="0 0 0"/>
     <geometry>
-      <mesh filename="package://URDF_description/meshes/base_link.stl" scale="0.001 0.001 0.001"/>
+      <mesh filename="package://my_bot/meshes/base_link.stl" scale="0.001 0.001 0.001"/>
     </geometry>
   </collision>
@@ -33,5 +33,5 @@
     <origin xyz="-0.101262 0.67433 -0.228037" rpy="0 0 0"/>
     <geometry>
-      <mesh filename="package://URDF_description/meshes/Bogie2_1.stl" scale="0.001 0.001 0.001"/>
+      <mesh filename="package://my_bot/meshes/Bogie2_1.stl" scale="0.001 0.001 0.001"/>
     </geometry>
     <material name="silver"/>
@@ -40,5 +40,5 @@
     <origin xyz="-0.101262 0.67433 -0.228037" rpy="0 0 0"/>
     <geometry>
-      <mesh filename="package://URDF_description/meshes/Bogie2_1.stl" scale="0.001 0.001 0.001"/>
+      <mesh filename="package://my_bot/meshes/Bogie2_1.stl" scale="0.001 0.001 0.001"/>
     </geometry>
   </collision>
@@ -53,5 +53,5 @@
     <origin xyz="-0.342141 0.375854 -0.3869" rpy="0 0 0"/>
     <geometry>
-      <mesh filename="package://URDF_description/meshes/Diff1_1.stl" scale="0.001 0.001 0.001"/>
+      <mesh filename="package://my_bot/meshes/Diff1_1.stl" scale="0.001 0.001 0.001"/>
     </geometry>
     <material name="silver"/>
@@ -60,5 +60,5 @@
     <origin xyz="-0.342141 0.375854 -0.3869" rpy="0 0 0"/>
     <geometry>
-      <mesh filename="package://URDF_description/meshes/Diff1_1.stl" scale="0.001 0.001 0.001"/>
+      <mesh filename="package://my_bot/meshes/Diff1_1.stl" scale="0.001 0.001 0.001"/>
     </geometry>
   </collision>
@@ -73,5 +73,5 @@
     <origin xyz="-0.488102 0.122014 -0.207048" rpy="0 0 0"/>
     <geometry>
-      <mesh filename="package://URDF_description/meshes/Bar1_1.stl" scale="0.001 0.001 0.001"/>
+      <mesh filename="package://my_bot/meshes/Bar1_1.stl" scale="0.001 0.001 0.001"/>
     </geometry>
     <material name="silver"/>
@@ -80,9 +80,9 @@
     <origin xyz="-0.488102 0.122014 -0.207048" rpy="0 0 0"/>
     <geometry>
-      <mesh filename="package://URDF_description/meshes/Bar1_1.stl" scale="0.001 0.001 0.001"/>
-    </geometry>
-  </collision>
-</link>
-<link name="Bar1_1">
+      <mesh filename="package://my_bot/meshes/Bar1_1.stl" scale="0.001 0.001 0.001"/>
+    </geometry>
+  </collision>
+</link>
+<link name="Bar1_2">
   <inertial>
     <origin xyz="-0.0453511772266767 0.03284580073433602 -0.08401395292890351" rpy="0 0 0"/>
@@ -93,5 +93,5 @@
     <origin xyz="-0.578805 0.187706 -0.375076" rpy="0 0 0"/>
     <geometry>
-      <mesh filename="package://URDF_description/meshes/Bar1_1.stl" scale="0.001 0.001 0.001"/>
+      <mesh filename="package://my_bot/meshes/Bar1_1.stl" scale="0.001 0.001 0.001"/>
     </geometry>
     <material name="silver"/>
@@ -100,5 +100,5 @@
     <origin xyz="-0.578805 0.187706 -0.375076" rpy="0 0 0"/>
     <geometry>
-      <mesh filename="package://URDF_description/meshes/Bar1_1.stl" scale="0.001 0.001 0.001"/>
+      <mesh filename="package://my_bot/meshes/Bar1_1.stl" scale="0.001 0.001 0.001"/>
     </geometry>
   </collision>
@@ -113,5 +113,5 @@
     <origin xyz="0.025606 0.447036 -0.394807" rpy="0 0 0"/>
     <geometry>
-      <mesh filename="package://URDF_description/meshes/Bar2_1.stl" scale="0.001 0.001 0.001"/>
+      <mesh filename="package://my_bot/meshes/Bar2_1.stl" scale="0.001 0.001 0.001"/>
     </geometry>
     <material name="silver"/>
@@ -120,9 +120,9 @@
     <origin xyz="0.025606 0.447036 -0.394807" rpy="0 0 0"/>
     <geometry>
-      <mesh filename="package://URDF_description/meshes/Bar2_1.stl" scale="0.001 0.001 0.001"/>
-    </geometry>
-  </collision>
-</link>
-<link name="Bar2_1">
+      <mesh filename="package://my_bot/meshes/Bar2_1.stl" scale="0.001 0.001 0.001"/>
+    </geometry>
+  </collision>
+</link>
+<link name="Bar2_2">
   <inertial>
     <origin xyz="-0.07413348749137935 0.0685212357582855 0.0017187497326043855" rpy="0 0 0"/>
@@ -133,5 +133,5 @@
     <origin xyz="-0.122661 0.584079 -0.39137" rpy="0 0 0"/>
     <geometry>
-      <mesh filename="package://URDF_description/meshes/Bar2_1.stl" scale="0.001 0.001 0.001"/>
+      <mesh filename="package://my_bot/meshes/Bar2_1.stl" scale="0.001 0.001 0.001"/>
     </geometry>
     <material name="silver"/>
@@ -140,5 +140,5 @@
     <origin xyz="-0.122661 0.584079 -0.39137" rpy="0 0 0"/>
     <geometry>
-      <mesh filename="package://URDF_description/meshes/Bar2_1.stl" scale="0.001 0.001 0.001"/>
+      <mesh filename="package://my_bot/meshes/Bar2_1.stl" scale="0.001 0.001 0.001"/>
     </geometry>
   </collision>
@@ -153,5 +153,5 @@
     <origin xyz="-0.069209 -0.367744 -0.38741" rpy="0 0 0"/>
     <geometry>
-      <mesh filename="package://URDF_description/meshes/Wheel1_1.stl" scale="0.001 0.001 0.001"/>
+      <mesh filename="package://my_bot/meshes/Wheel1_1.stl" scale="0.001 0.001 0.001"/>
     </geometry>
     <material name="silver"/>
@@ -160,5 +160,5 @@
     <origin xyz="-0.069209 -0.367744 -0.38741" rpy="0 0 0"/>
     <geometry>
-      <mesh filename="package://URDF_description/meshes/Wheel1_1.stl" scale="0.001 0.001 0.001"/>
+      <mesh filename="package://my_bot/meshes/Wheel1_1.stl" scale="0.001 0.001 0.001"/>
     </geometry>
   </collision>
@@ -173,5 +173,5 @@
     <origin xyz="-0.230521 -0.22289 -0.14374" rpy="0 0 0"/>
     <geometry>
-      <mesh filename="package://URDF_description/meshes/Wheel2_1.stl" scale="0.001 0.001 0.001"/>
+      <mesh filename="package://my_bot/meshes/Wheel2_1.stl" scale="0.001 0.001 0.001"/>
     </geometry>
     <material name="silver"/>
@@ -180,5 +180,5 @@
     <origin xyz="-0.230521 -0.22289 -0.14374" rpy="0 0 0"/>
     <geometry>
-      <mesh filename="package://URDF_description/meshes/Wheel2_1.stl" scale="0.001 0.001 0.001"/>
+      <mesh filename="package://my_bot/meshes/Wheel2_1.stl" scale="0.001 0.001 0.001"/>
     </geometry>
   </collision>
@@ -193,5 +193,5 @@
     <origin xyz="-0.143367 -0.225919 0.163611" rpy="0 0 0"/>
     <geometry>
-      <mesh filename="package://URDF_description/meshes/Wheel3_1.stl" scale="0.001 0.001 0.001"/>
+      <mesh filename="package://my_bot/meshes/Wheel3_1.stl" scale="0.001 0.001 0.001"/>
     </geometry>
     <material name="silver"/>
@@ -200,5 +200,5 @@
     <origin xyz="-0.143367 -0.225919 0.163611" rpy="0 0 0"/>
     <geometry>
-      <mesh filename="package://URDF_description/meshes/Wheel3_1.stl" scale="0.001 0.001 0.001"/>
+      <mesh filename="package://my_bot/meshes/Wheel3_1.stl" scale="0.001 0.001 0.001"/>
     </geometry>
   </collision>
@@ -213,5 +213,5 @@
     <origin xyz="0.291017 0.34301 0.210668" rpy="0 0 0"/>
     <geometry>
-      <mesh filename="package://URDF_description/meshes/Wheel4_1.stl" scale="0.001 0.001 0.001"/>
+      <mesh filename="package://my_bot/meshes/Wheel4_1.stl" scale="0.001 0.001 0.001"/>
     </geometry>
     <material name="silver"/>
@@ -220,5 +220,5 @@
     <origin xyz="0.291017 0.34301 0.210668" rpy="0 0 0"/>
     <geometry>
-      <mesh filename="package://URDF_description/meshes/Wheel4_1.stl" scale="0.001 0.001 0.001"/>
+      <mesh filename="package://my_bot/meshes/Wheel4_1.stl" scale="0.001 0.001 0.001"/>
     </geometry>
   </collision>
@@ -233,5 +233,5 @@
     <origin xyz="-0.275576 0.947443 -0.074581" rpy="0 0 0"/>
     <geometry>
-      <mesh filename="package://URDF_description/meshes/Wheel5_1.stl" scale="0.001 0.001 0.001"/>
+      <mesh filename="package://my_bot/meshes/Wheel5_1.stl" scale="0.001 0.001 0.001"/>
     </geometry>
     <material name="silver"/>
@@ -240,5 +240,5 @@
     <origin xyz="-0.275576 0.947443 -0.074581" rpy="0 0 0"/>
     <geometry>
-      <mesh filename="package://URDF_description/meshes/Wheel5_1.stl" scale="0.001 0.001 0.001"/>
+      <mesh filename="package://my_bot/meshes/Wheel5_1.stl" scale="0.001 0.001 0.001"/>
     </geometry>
   </collision>
@@ -253,5 +253,5 @@
     <origin xyz="-0.322519 0.906694 -0.387959" rpy="0 0 0"/>
     <geometry>
-      <mesh filename="package://URDF_description/meshes/Wheel6_1.stl" scale="0.001 0.001 0.001"/>
+      <mesh filename="package://my_bot/meshes/Wheel6_1.stl" scale="0.001 0.001 0.001"/>
     </geometry>
     <material name="silver"/>
@@ -260,5 +260,5 @@
     <origin xyz="-0.322519 0.906694 -0.387959" rpy="0 0 0"/>
     <geometry>
-      <mesh filename="package://URDF_description/meshes/Wheel6_1.stl" scale="0.001 0.001 0.001"/>
+      <mesh filename="package://my_bot/meshes/Wheel6_1.stl" scale="0.001 0.001 0.001"/>
     </geometry>
   </collision>
@@ -273,5 +273,5 @@
     <origin xyz="-0.372144 0.031872 0.064979" rpy="0 0 0"/>
     <geometry>
-      <mesh filename="package://URDF_description/meshes/Bogie4_1.stl" scale="0.001 0.001 0.001"/>
+      <mesh filename="package://my_bot/meshes/Bogie4_1.stl" scale="0.001 0.001 0.001"/>
     </geometry>
     <material name="silver"/>
@@ -280,5 +280,5 @@
     <origin xyz="-0.372144 0.031872 0.064979" rpy="0 0 0"/>
     <geometry>
-      <mesh filename="package://URDF_description/meshes/Bogie4_1.stl" scale="0.001 0.001 0.001"/>
+      <mesh filename="package://my_bot/meshes/Bogie4_1.stl" scale="0.001 0.001 0.001"/>
     </geometry>
   </collision>
@@ -293,5 +293,5 @@
     <origin xyz="-0.392766 0.076779 -0.180422" rpy="0 0 0"/>
     <geometry>
-      <mesh filename="package://URDF_description/meshes/Bogie3_1.stl" scale="0.001 0.001 0.001"/>
+      <mesh filename="package://my_bot/meshes/Bogie3_1.stl" scale="0.001 0.001 0.001"/>
     </geometry>
     <material name="silver"/>
@@ -300,5 +300,5 @@
     <origin xyz="-0.392766 0.076779 -0.180422" rpy="0 0 0"/>
     <geometry>
-      <mesh filename="package://URDF_description/meshes/Bogie3_1.stl" scale="0.001 0.001 0.001"/>
+      <mesh filename="package://my_bot/meshes/Bogie3_1.stl" scale="0.001 0.001 0.001"/>
     </geometry>
   </collision>
@@ -313,5 +313,5 @@
     <origin xyz="0.002504 0.454759 -0.288737" rpy="0 0 0"/>
     <geometry>
-      <mesh filename="package://URDF_description/meshes/Bogie1_1.stl" scale="0.001 0.001 0.001"/>
+      <mesh filename="package://my_bot/meshes/Bogie1_1.stl" scale="0.001 0.001 0.001"/>
     </geometry>
     <material name="silver"/>
@@ -320,5 +320,5 @@
     <origin xyz="0.002504 0.454759 -0.288737" rpy="0 0 0"/>
     <geometry>
-      <mesh filename="package://URDF_description/meshes/Bogie1_1.stl" scale="0.001 0.001 0.001"/>
+      <mesh filename="package://my_bot/meshes/Bogie1_1.stl" scale="0.001 0.001 0.001"/>
     </geometry>
   </collision>
@@ -342,8 +342,9 @@
   <axis xyz="0.699606 -0.64133 0.315035"/>
 </joint>
+<!-- one of these two may need to swicth-->
 <joint name="Revolute 7" type="continuous">
   <origin xyz="0.236664 0.188148 -0.011824" rpy="0 0 0"/>
   <parent link="Diff1_1"/>
-  <child link="Bar1_1"/>
+  <child link="Bar1_2"/>
   <axis xyz="0.626432 -0.731916 -0.268109"/>
 </joint>
@@ -354,8 +355,9 @@
   <axis xyz="0.005692 -0.280968 -0.9597"/>
 </joint>
+<!-- one of these two may need to swicth-->
 <joint name="Revolute 9" type="continuous">
   <origin xyz="-0.21948 -0.208225 0.00447" rpy="0 0 0"/>
   <parent link="Diff1_1"/>
-  <child link="Bar2_1"/>
+  <child link="Bar2_2"/>
   <axis xyz="0.626432 -0.731916 -0.268109"/>
 </joint>

Commit message: added mass to the bass link cause mass can not equal 0

File: description/robot.urdf.xacro (robot description, xacro)
@@ -7,5 +7,5 @@
   <inertial>
     <origin xyz="0.0 0.0 0.0" rpy="0 0 0"/>
-    <mass value="0.0"/>
+    <mass value="0.00001"/>
     <inertia ixx="0.0" iyy="0.0" izz="0.0" ixy="0.0" iyz="0.0" ixz="0.0"/>
   </inertial>

Commit message: inertia was too negligable

File: description/robot.urdf.xacro (robot description, xacro)
@@ -7,6 +7,6 @@
   <inertial>
     <origin xyz="0.0 0.0 0.0" rpy="0 0 0"/>
-    <mass value="0.00001"/>
-    <inertia ixx="0.00001" iyy="0.00001" izz="0.00001" ixy="0.00001" iyz="0.00001" ixz="0.00001"/>
+    <mass value="0.01"/>
+    <inertia ixx="0.01" iyy="0.01" izz="0.01" ixy="0.01" iyz="0.01" ixz="0.01"/>
   </inertial>
   <visual>

Commit message: inertia still too small

File: description/robot.urdf.xacro (robot description, xacro)
@@ -8,5 +8,5 @@
     <origin xyz="0.0 0.0 0.0" rpy="0 0 0"/>
     <mass value="0.01"/>
-    <inertia ixx="0.01" iyy="0.01" izz="0.01" ixy="0.01" iyz="0.01" ixz="0.01"/>
+    <inertia ixx="0.1" iyy="0.1" izz="0.1" ixy="0" iyz="0" ixz="0"/>
   </inertial>
   <visual>

Commit message: adjusted child referneces

File: description/robot.urdf.xacro (robot description, xacro)
@@ -339,5 +339,5 @@
   <origin xyz="0.186039 -0.110927 0.194654" rpy="0 0 0"/>
   <parent link="Bogie3_1"/>
-  <child link="Bar1_1"/>
+  <child link="Bar1_2"/>
   <axis xyz="0.699606 -0.64133 0.315035"/>
 </joint>
@@ -346,5 +346,5 @@
   <origin xyz="0.236664 0.188148 -0.011824" rpy="0 0 0"/>
   <parent link="Diff1_1"/>
-  <child link="Bar1_2"/>
+  <child link="Bar1_1"/>
   <axis xyz="0.626432 -0.731916 -0.268109"/>
 </joint>
@@ -352,5 +352,5 @@
   <origin xyz="0.125165 -0.12932 0.102633" rpy="0 0 0"/>
   <parent link="Bogie1_1"/>
-  <child link="Bar2_1"/>
+  <child link="Bar2_2"/>
   <axis xyz="0.005692 -0.280968 -0.9597"/>
 </joint>
@@ -359,5 +359,5 @@
   <origin xyz="-0.21948 -0.208225 0.00447" rpy="0 0 0"/>
   <parent link="Diff1_1"/>
-  <child link="Bar2_2"/>
+  <child link="Bar2_1"/>
   <axis xyz="0.626432 -0.731916 -0.268109"/>
 </joint>

Commit message: changed yaml file

File: description/robot.urdf.xacro (robot description, xacro)
@@ -339,5 +339,5 @@
   <origin xyz="0.186039 -0.110927 0.194654" rpy="0 0 0"/>
   <parent link="Bogie3_1"/>
-  <child link="Bar1_2"/>
+  <child link="Bar1_1"/>
   <axis xyz="0.699606 -0.64133 0.315035"/>
 </joint>
@@ -346,5 +346,5 @@
   <origin xyz="0.236664 0.188148 -0.011824" rpy="0 0 0"/>
   <parent link="Diff1_1"/>
-  <child link="Bar1_1"/>
+  <child link="Bar1_2"/>
   <axis xyz="0.626432 -0.731916 -0.268109"/>
 </joint>
@@ -352,5 +352,5 @@
   <origin xyz="0.125165 -0.12932 0.102633" rpy="0 0 0"/>
   <parent link="Bogie1_1"/>
-  <child link="Bar2_2"/>
+  <child link="Bar2_1"/>
   <axis xyz="0.005692 -0.280968 -0.9597"/>
 </joint>
@@ -359,5 +359,5 @@
   <origin xyz="-0.21948 -0.208225 0.00447" rpy="0 0 0"/>
   <parent link="Diff1_1"/>
-  <child link="Bar2_1"/>
+  <child link="Bar2_2"/>
   <axis xyz="0.626432 -0.731916 -0.268109"/>
 </joint>
